File: ModernVtwin.brd (EAGLE design)
At the start: 160 x 147 mm, 152 parts, among them IC1 TL072P, IC2 TL071P, IC3 TL072P, IC4 TL072P, IC5 7812TV, IC7 PIC16F57, IC8 7805T, Q1 J175, Q2 J175, Q3 J175, Q4 J175, Q5 J175, Q6 J175, Q7 J175, Q8 J175, T1_P35(B)_TOEI_TRANS POWERTRANS_FOR_VALVE

Commit message: no message
Parts:
- moved C1 149.9 mm to (-64.8, 68.6)
- moved C10 149.9 mm to (-102.9, 68.6)
- moved C12 149.9 mm to (-118.1, 68.6)
- moved C14 149.9 mm to (-24.1, 78.7)
- moved C15 149.9 mm to (-31.8, 78.7)
- moved C17 149.9 mm to (-74.9, 94.0)
- moved C18 149.9 mm to (-47.0, 78.7)
- moved C19 149.9 mm to (-54.6, 78.7)
- moved C21 149.9 mm to (-81.3, 94.0)
- moved C22 149.9 mm to (-69.8, 78.7)
- moved C23 149.9 mm to (-77.5, 78.7)
- moved C25 149.9 mm to (-85.1, 78.7)
- moved C27 149.9 mm to (-29.2, 94.0)
- moved C28 149.9 mm to (-38.1, 94.0)
- moved C29 149.9 mm to (-47.0, 94.0)
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Connections:
- net N$100 renamed Q3
- removed net N$101: D11.C
- removed net N$102: D12.C
- removed net N$103: D13.C
- removed net N$104: D14.C
- removed net N$105: D15.C
- removed net N$107: Q7.G
- removed net N$2: Q1.G
- removed net N$34: Q8.G
- removed net N$48: Q6.G
- removed net N$60: Q4.G
- removed net N$7: Q2.G
- removed net N$91: D8.C
- removed net N$99: D9.C
- new net Q1: D8.C, Q1.G
- new net Q2: D9.C, Q2.G
- new net Q4: D11.C, Q4.G
- new net Q6: D13.C, Q6.G
- new net Q7: D14.C, Q7.G
- new net Q8: D15.C, Q8.G
- net Q5: now also D12.C
Other:
- board size 160 x 147 mm -> 160 x 100 mm
