File: ModernVtwin.sch (EAGLE design)
At the start: 152 parts, among them IC1 TL072P, IC2 TL071P, IC3 TL072P, IC4 TL072P, IC5 7812TV, IC7 PIC16F57, IC8 7805T, Q1 J175, Q2 J175, Q3 J175, Q4 J175, Q5 J175, Q6 J175, Q7 J175, Q8 J175

Commit message: no message
Parts:
- removed U$1: POWERTRANS_FOR_VALVE, transformer-pulse:POWERTRANS_FOR_VALVE
- added T1_P35(B)_TOEI_TRANS: POWERTRANS_FOR_VALVE, transformer-pulse:POWERTRANS_FOR_VALVE
- C27, C28, C29, C30: value 15u -> 10u350V
- C31, C32: value 15u -> 1000u 25V
- C33, C34, C35, C46: value 15u -> 1000u25V
- C47: value 103 -> 270nF
- C48: value 103 -> 270n
- R44: value 1.5k -> 1M
- R45, R46, R47: value 1.5k -> 4k7
- R48: value 1.5k -> 2.7R5W
Connections:
- net N$100 renamed Q3
- removed net N$101: D11.C
- removed net N$102: D12.C
- removed net N$103: D13.C
- removed net N$104: D14.C
- removed net N$105: D15.C
- removed net N$107: Q7.G
- removed net N$2: Q1.G
- removed net N$34: Q8.G
- removed net N$48: Q6.G
- removed net N$60: Q4.G
- removed net N$7: Q2.G
- removed net N$91: D8.C
- removed net N$99: D9.C
- new net Q1: D8.C, Q1.G
- new net Q2: D9.C, Q2.G
- new net Q4: D11.C, Q4.G
- new net Q6: D13.C, Q6.G
- new net Q7: D14.C, Q7.G
- new net Q8: D15.C, Q8.G
- net +5V: now also T1_P35(B)_TOEI_TRANS.VH2+
- net -12V: now also C46.2; no longer C46.1
- net GND: now also C34.1, C46.1, T1_P35(B)_TOEI_TRANS.VH-, T1_P35(B)_TOEI_TRANS.VH2-; no longer C34.2, C46.2
- net N$111: now also T1_P35(B)_TOEI_TRANS.VB-
- net N$116: now also C34.2; no longer C34.1
- net N$59: now also T1_P35(B)_TOEI_TRANS.100VIN+; no longer U$1.100VIN+
- net N$62: now also T1_P35(B)_TOEI_TRANS.100VIN-; no longer U$1.100VIN-
- net N$65: now also T1_P35(B)_TOEI_TRANS.VB+
- net N$66: now also T1_P35(B)_TOEI_TRANS.VH+
- net Q5: now also D12.C
Other:
- note added: "These 12V for OpAmps"
- moved on the sheet: C27, C28, C29, C30, C31, C32, C33, C34, C35, C36, C37, C38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
